File: projects/20241128-servo/kicad-schematics/schema.kicad_sch (KiCad schematic)
At the start: 2 parts, among them M1 Motor_Servo, SW1 SW_Push

Commit message: update schema
Parts:
- added BT1: 4x AA, symbol Device:Battery_Cell
- M1: value Motor_Servo -> SG90/MG90S
Connections:
- net GND: now also BT1.2 (-)
- net 4x AA: no longer names the net of M1.2 (+)
- net 4x AA: now also BT1.1 (+)
Other:
- moved on the sheet: M1, SW1
